File: totpvault-hardware/totpvault-hardware.kicad_pcb (KiCad board)
At the start: 2 copper layers, 15 x 40 mm, 30 parts, among them J2 Conn_01x04_Socket, J3 Conn_01x02_Socket, P1 USB_C_Plug, U1 ESP32-C3, U3 CH343P, U4 USBLC6-2SC6, U5 HT75xx-1-SOT89, Y1 Crystal_GND24

Commit message: PCB order
Parts:
- removed P1: USB_C_Plug, Connector_USB:USB_C_Plug_Molex_105444
- removed R1: 5.1k, Resistor_SMD:R_0603_1608Metric
- added X16: ~, Misc:USB_C_Connector, F.Cu at (108.4, 69.1)
- moved C15 0.20 mm to (105.1, 96.5)
Connections:
- U4 pad 4: Net-(P1-D+) -> /D+
- U4 pad 6: Net-(P1-D-) -> /D-
Routing:
- net VBUS: track 55.0 -> 44.9 mm, vias 4 -> 5
- net Net-(P1-D-): track 9.13 -> 0.00 mm
- net /D-: track 0.00 -> 8.40 mm
- net /D+: track 0.00 -> 8.35 mm
- net Net-(P1-CC): track 7.32 -> 0.00 mm
- net Net-(P1-D+): track 6.29 -> 0.00 mm, vias 2 -> 0
- net GND: track 73.9 -> 69.0 mm, vias 25 -> 23
