File: totpvault-hardware/totpvault-hardware.kicad_sch (KiCad schematic)
At the start: 29 parts, among them J2 Conn_01x04_Socket, J3 Conn_01x02_Socket, P1 USB_C_Plug, U1 ESP32-C3, U3 CH343P, U4 USBLC6-2SC6, U5 HT75xx-1-SOT89, Y1 Crystal_GND24

Commit message: PCB order
Parts:
- removed P1: USB_C_Plug, Connector_USB:USB_C_Plug_Molex_105444, symbol Connector:USB_C_Plug
- removed R1: 5.1k, Resistor_SMD:R_0603_1608Metric, symbol Device:R
- added X16: ~, Misc:USB_C_Connector, symbol Misc:USB_C_Connector
Connections:
- net GND: now also X16.4 (GND)
- net VBUS: now also X16.1 (VBUS)
- net D+: now reaches U4.4 (I/O2)
- net D+: now also X16.3 (D+)
- net D-: now reaches U4.6 (I/O1)
- net D-: now also X16.2 (D-)
- no-connect marks 36 -> 25
